Commit message: tested the mobile manipulator code failed

File: ompl_test/urdf/agv.urdf (robot description, URDF)
Before this commit: robot agv, 1 links, 0 joints
Links:
- added link arm_link_1; visual box size=0.2 0.05 0.05
Joints:
- added joint base_arm: type revolute, parent base_link, child arm_link_1, origin xyz=0.0 0.0 0.05, axis 0 0 1, limit lower=-3.14 upper=3.14 effort=300 velocity=0.1
