Commit message: changed the environment obstacle to smaller ones

File: ompl_test/urdf/ur10.urdf (robot description, URDF)
Before this commit: robot mobile_manipulator, 10 links, 9 joints
Links:
- link base_link: geometry collision mesh filename=package://ur_e_description/meshes/ur10e/collision/base.dae; visual mesh filename=package://ur_e_description/meshes/ur10e/visual/base.dae
- link forearm_link: geometry collision mesh filename=package://ur_e_description/meshes/ur10e/collision/forearm.d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; visual mesh filename=package://ur_e_description/meshes/ur10e/visual/forearm.dae
- link shoulder_link: geometry collision mesh filename=package://ur_e_description/meshes/ur10e/collision/shoulder.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; visual mesh filename=package://ur_e_description/meshes/ur10e/visual/shoulder.dae
- link upper_arm_link: geometry collision mesh filename=package://ur_e_description/meshes/ur10e/collision/upperarm.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; visual mesh filename=package://ur_e_description/meshes/ur10e/visual/upperarm.dae
- link wrist_1_link: geometry collision mesh filename=package://ur_e_description/meshes/ur10e/collision/wrist1.dae; visual mesh filename=package://ur_e_description/meshes/ur10e/visual/wrist1.dae
- link wrist_2_link: geometry collision mesh filename=package://ur_e_description/meshes/ur10e/collision/wrist2.dae; visual mesh filename=package://ur_e_description/meshes/ur10e/visual/wrist2.dae
- link wrist_3_link: geometry collision mesh filename=package://ur_e_description/meshes/ur10e/collision/wrist3.dae; visual mesh filename=package://ur_e_description/meshes/ur10e/visual/wrist3.dae
